Commit message: Changed urdfs for single moteus test

File: test/urdf/core/single_joint.urdf.xacro (robot description, xacro)
@@ -22,7 +22,4 @@
         </visual>
     </link>
-    <gazebo reference="${name}_stator">
-        <material>Gazebo/Red</material>
-    </gazebo>
     <link name="${name}_rotor">
         <inertial>
@@ -50,7 +47,4 @@
         </visual>
     </link>
-    <gazebo reference="${name}_rotor">
-        <material>Gazebo/Green</material>
-    </gazebo>
     <joint name="${parent_name}_${name}" type="fixed">
         <origin xyz="${x} ${y} ${stator_length/2}" rpy="0.0 0.0 0.0"/>

File: test/urdf/test_single_moteus.urdf.xacro (robot description, xacro)
@@ -9,5 +9,5 @@
     <!-- Single joint macro -->
     <xacro:include filename="core/single_joint.urdf.xacro"/>
-    <link name="world" />
+    <link name="world"/>
     <xacro:single_joint_macro name="actuator_1" parent_name="world" x="0.0" y="0.0" inertia="${rotor_inertia}" pos_max="${motor_position_max}" pos_min="${motor_position_min}" vel_max="${motor_velocity_max}" effort_max="${motor_effort_max}"/>
     <ros2_control name="pi3hat_hardware_interface" type="system">
@@ -17,5 +17,5 @@
             <param name="imu_mounting_deg.pitch">0</param>
             <param name="imu_mounting_deg.roll">0</param>
-            <param name="imu_sampling_rate">1000</param>
+            <param name="imu_sampling_rate">100</param>
             <param name="can_1_fdcan_frame">true</param>
             <param name="can_1_automatic_retransmission">true</param>
