Commit message: Modified single motor test

File: test/urdf/test_single_moteus.urdf.xacro (robot description, xacro)
@@ -1,51 +1,14 @@
 <?xml version="1.0"?>
 <robot xmlns:xacro="http://www.ros.org/wiki/xacro" name="test_single_moteus">
-  <link name="box">
-        <visual>
-            <origin xyz="0.0 0.0 0.0" rpy="0.0 0.0 0.0"/>
-            <geometry>
-                <box size="0.5 0.5 0.5"/>
-            </geometry>
-            <material name="red">
-                <color rgba="1.0 0.0 0.0 1.0"/>
-            </material>
-        </visual>
-    </link>
-    <link name="rotor">
-        <visual>
-            <origin xyz="0.0 0.0 0.0" rpy="0.0 0.0 0.0"/>
-            <geometry>
-                <cylinder radius="0.2" length="0.1"/>
-            </geometry>
-            <material name="red">
-                <color rgba="0.0 0.0 1.0 1.0"/>
-            </material>
-        </visual>
-    </link>
-    <link name="indicator">
-        <visual>
-            <origin xyz="0.0 0.0 0.0" rpy="0.0 0.0 0.0"/>
-            <geometry>
-                <box size="0.01 0.3 0.01"/>
-            </geometry>
-            <material name="">
-                <color rgba="0.0 1.0 0.0 1.0"/>
-                <texture filename=""/>
-            </material>
-        </visual>
-    </link>
-    <joint name="joint_1" type="revolute">
-        <origin xyz="0.0 0.3 0.0" rpy="-1.5707 0.0 0.0"/>
-        <parent link="box"/>
-        <child link="rotor"/>
-        <axis xyz="0.0 0.0 -1.0"/>
-        <limit lower="-10.0" upper="10.0" effort="10.0" velocity="100.0"/>
-    </joint>
-    <joint name="joint_2" type="fixed">
-        <origin xyz="0.0 -0.25 0.055" rpy="0.0 0.0 0.0"/>
-        <parent link="rotor"/>
-        <child link="indicator"/>
-    </joint>
-  <ros2_control name="pi3hat_hardware_interface" type="system">
+    <xacro:property name="PI" value="3.141592"/>
+    <xacro:property name="rotor_inertia" value="1.0"/>
+    <xacro:property name="motor_position_max" value="${10 * PI}"/>
+    <xacro:property name="motor_position_min" value="${-10 * PI}"/>
+    <xacro:property name="motor_velocity_max" value="10.0"/>
+    <xacro:property name="motor_effort_max" value="0.2"/>
+    <!-- Single joint macro -->
+    <xacro:include filename="core/single_joint.urdf.xacro"/>
+    <xacro:single_joint_macro name="actuator_1" parent_name="world" x="0.0" y="0.0" inertia="${rotor_inertia}" pos_max="${motor_position_max}" pos_min="${motor_position_min}" vel_max="${motor_velocity_max}" effort_max="${motor_effort_max}"/>
+    <ros2_control name="pi3hat_hardware_interface" type="system">
         <hardware>
             <plugin>pi3hat_hardware_interface/Pi3HatHardwareInterface</plugin>
@@ -70,30 +33,15 @@
             <param name="can_5_bitrate_switch">true</param>
         </hardware>
-        <joint name="joint_1">
-            <param name="controller_type">moteus</param>
-            <param name="controller_can_bus">1</param>
-            <param name="controller_can_id">1</param>
-            <param name="motor_direction">1</param>
-            <param name="motor_position_offset">0.0</param>
-            <param name="motor_position_max">500.0</param>
-            <param name="motor_position_min">-500.0</param>
-            <param name="motor_velocity_max">10.0</param>
-            <param name="motor_torque_max">0.2</param>
-            <command_interface name="position"/>
-            <command_interface name="velocity"/>
-            <command_interface name="effort"/>
-            <state_interface name="position"/>
-            <state_interface name="velocity"/>
-            <state_interface name="effort"/>
-            <state_interface name="temperature"/>
-      </joint>
-    <transmission name="transmission1">
-        <plugin>transmission_interface/SimpleTransmission</plugin>
-        <actuator name="actuator_1" role="actuator1"/>
-        <joint name="joint_1" role="joint1">
-            <mechanical_reduction>16.0</mechanical_reduction>
-            <offset>0.0</offset>
-        </joint>
-    </transmission>
+        <!-- Single motor hardware macro -->
+        <xacro:include filename="core/single_motor_hardware.urdf.xacro"/>
+        <xacro:single_motor_hardware_macro name="actuator_1" type="moteus" can_bus="1" can_id="1" direction="1" offset="0.0" pos_max="${motor_position_max}" pos_min="${motor_position_min}" vel_max="${motor_velocity_max}" torque_max="${motor_effort_max}"/>
+        <!-- <transmission name="transmission1">
+            <plugin>transmission_interface/SimpleTransmission</plugin>
+            <actuator name="actuator_1" role="actuator1"/>
+            <joint name="joint_1" role="joint1">
+                <mechanical_reduction>16.0</mechanical_reduction>
+                <offset>0.0</offset>
+            </joint>
+        </transmission> -->
       <sensor name="imu_sensor">
           <state_interface name="orientation.x"/>

Commit message: Fixed single test example

File: test/urdf/test_single_moteus.urdf.xacro (robot description, xacro)
@@ -7,8 +7,11 @@
     <xacro:property name="motor_velocity_max" value="2.0"/>
     <xacro:property name="motor_effort_max" value="0.2"/>
+    <xacro:property name="transmission_reduction" value="9.97"/>
+    <xacro:property name="transmission_offset" value="0.0"/>
     <!-- Single joint macro -->
     <xacro:include filename="core/single_joint.urdf.xacro"/>
     <link name="world"/>
     <xacro:single_joint_macro name="actuator_1" parent_name="world" x="0.0" y="0.0" inertia="${rotor_inertia}" pos_max="${motor_position_max}" pos_min="${motor_position_min}" vel_max="${motor_velocity_max}" effort_max="${motor_effort_max}"/>
+    <!-- Hardware interface for pi3hat -->
     <ros2_control name="pi3hat_hardware_interface" type="system">
         <hardware>
@@ -37,24 +40,19 @@
         <xacro:include filename="core/single_motor_hardware.urdf.xacro"/>
         <xacro:single_motor_hardware_macro name="actuator_1" type="moteus" can_bus="1" can_id="2" direction="1" offset="0.0" pos_max="${motor_position_max}" pos_min="${motor_position_min}" vel_max="${motor_velocity_max}" torque_max="${motor_effort_max}"/>
-        <!-- <transmission name="transmission1">
-            <plugin>transmission_interface/SimpleTransmission</plugin>
-            <actuator name="actuator_1" role="actuator1"/>
-            <joint name="joint_1" role="joint1">
-                <mechanical_reduction>10.0</mechanical_reduction>
-                <offset>0.0</offset>
-            </joint>
-        </transmission> -->
-      <sensor name="imu_sensor">
-          <state_interface name="orientation.x"/>
-          <state_interface name="orientation.y"/>
-          <state_interface name="orientation.z"/>
-          <state_interface name="orientation.w"/>
-          <state_interface name="angular_velocity.x"/>
-          <state_interface name="angular_velocity.y"/>
-          <state_interface name="angular_velocity.z"/>
-          <state_interface name="linear_acceleration.x"/>
-          <state_interface name="linear_acceleration.y"/>
-          <state_interface name="linear_acceleration.z"/>
-      </sensor>
-  </ros2_control>
+        <!-- Simple transmission macro -->
+        <xacro:include filename="core/simple_transmission_macro.urdf.xacro"/>
+        <xacro:simple_transmission_macro transmission_name="transmission_1" actuator_name="actuator_1" joint_name="actuator_1_joint" reduction="${transmission_reduction}" offset="${transmission_offset}"/>
+        <sensor name="imu_sensor">
+            <state_interface name="orientation.x"/>
+            <state_interface name="orientation.y"/>
+            <state_interface name="orientation.z"/>
+            <state_interface name="orientation.w"/>
+            <state_interface name="angular_velocity.x"/>
+            <state_interface name="angular_velocity.y"/>
+            <state_interface name="angular_velocity.z"/>
+            <state_interface name="linear_acceleration.x"/>
+            <state_interface name="linear_acceleration.y"/>
+            <state_interface name="linear_acceleration.z"/>
+        </sensor>
+    </ros2_control>
 </robot>

Commit message: Init pos read/write on base motor

File: test/urdf/test_single_moteus.urdf.xacro (robot description, xacro)
@@ -3,14 +3,14 @@
     <xacro:property name="PI" value="3.141592"/>
     <xacro:property name="rotor_inertia" value="1.0"/>
-    <xacro:property name="motor_position_max" value="${10 * PI}"/>
-    <xacro:property name="motor_position_min" value="${-10 * PI}"/>
+    <xacro:property name="motor_position_max" value="${ PI * 9}"/>
+    <xacro:property name="motor_position_min" value="${-PI * 9}"/>
     <xacro:property name="motor_velocity_max" value="2.0"/>
     <xacro:property name="motor_effort_max" value="0.2"/>
-    <xacro:property name="transmission_reduction" value="9.97"/>
+    <xacro:property name="transmission_reduction" value="9.0"/>
     <xacro:property name="transmission_offset" value="0.0"/>
     <!-- Single joint macro -->
     <xacro:include filename="core/single_joint.urdf.xacro"/>
     <link name="world"/>
-    <xacro:single_joint_macro name="actuator_1" parent_name="world" x="0.0" y="0.0" inertia="${rotor_inertia}" pos_max="${motor_position_max}" pos_min="${motor_position_min}" vel_max="${motor_velocity_max}" effort_max="${motor_effort_max}"/>
+    <xacro:single_joint_macro name="actuator_5" parent_name="world" x="0.0" y="0.0" inertia="${rotor_inertia}" pos_max="${motor_position_max}" pos_min="${motor_position_min}" vel_max="${motor_velocity_max}" effort_max="${motor_effort_max}"/>
     <!-- Hardware interface for pi3hat -->
     <ros2_control name="pi3hat_hardware_interface" type="system">
@@ -39,8 +39,8 @@
         <!-- Single motor hardware macro -->
         <xacro:include filename="core/single_motor_hardware.urdf.xacro"/>
-        <xacro:single_motor_hardware_macro name="actuator_1" type="moteus" can_bus="1" can_id="2" direction="1" offset="0.0" pos_max="${motor_position_max}" pos_min="${motor_position_min}" vel_max="${motor_velocity_max}" torque_max="${motor_effort_max}"/>
+        <xacro:single_motor_hardware_macro name="actuator_5" type="moteus" can_bus="1" can_id="1" direction="1" offset="0.0" pos_max="${motor_position_max}" pos_min="${motor_position_min}" vel_max="${motor_velocity_max}" torque_max="${motor_effort_max}"/>
         <!-- Simple transmission macro -->
         <xacro:include filename="core/simple_transmission_macro.urdf.xacro"/>
-        <xacro:simple_transmission_macro transmission_name="transmission_1" actuator_name="actuator_1" joint_name="actuator_1_joint" reduction="${transmission_reduction}" offset="${transmission_offset}"/>
+        <xacro:simple_transmission_macro transmission_name="transmission_5" actuator_name="actuator_5" joint_name="actuator_5_joint" reduction="${transmission_reduction}" offset="${transmission_offset}"/>
         <sensor name="imu_sensor">
             <state_interface name="orientation.x"/>
