Commit message: Got basic differential to work!

File: test/urdf/myrobot.urdf.xacro (robot description, xacro)
@@ -4,9 +4,12 @@
 	<xacro:property name="reduc_9_actuator_diameter" value="${0.077 * multiplier}"/>
 	<xacro:property name="reduc_9_actuator_height" value="${0.058 * multiplier}"/>
+	<xacro:property name="waist_reduction_ratio" value="9"/>
 	<xacro:property name="waist_arm_height" value="${0.01 * multiplier}"/>
+	<xacro:property name="shoulder_reduction_ratio" value="9"/>
 	<xacro:property name="shoulder_arm_angle_offset" value="${-0.5*pi - 0.52/4.5*pi}"/>
 	<xacro:property name="shoulder_arm_length" value="${0.1385 * multiplier}"/>
 	<xacro:property name="shoulder_arm_width" value="${0.047 * multiplier}"/>
 	<xacro:property name="arm_height" value="${0.03 * multiplier}"/>
+	<xacro:property name="elbow_reduction_ratio" value="5"/>
 	<xacro:property name="elbow_arm1_angle_offset" value="${-pi/6 + 0.15/2.5*pi}"/>
 	<xacro:property name="elbow_arm2_angle_offset" value="-${pi/4}"/>
@@ -14,4 +17,5 @@
 	<xacro:property name="elbow_arm2_length" value="${0.110 * multiplier}"/>
 	<xacro:property name="elbow_arm_width" value="${0.020 * multiplier}"/>
+	<xacro:property name="wrist_reduction_ratio" value="6"/>
 	<xacro:property name="wrist_angle_offset" value="${-pi/4 - elbow_arm1_angle_offset}"/>
 	<xacro:property name="wrist_diameter" value="${0.04 * multiplier}"/>
@@ -146,8 +150,8 @@
 		</collision>
 	</link>
-	<link name="wrist">
-		<visual>
-			<geometry>
-				<cylinder length="${reduc_9_actuator_height/2}" radius="${wrist_diameter/2}" />
+	<link name="left_differential">
+		<visual>
+			<geometry>
+				<cylinder length="${reduc_9_actuator_height/8}" radius="${wrist_diameter/4}" />
 			</geometry>
 			<origin rpy="0 0 0" xyz="0 0 0"/>
@@ -156,20 +160,20 @@
 		<collision>
 			<geometry>
-				<cylinder length="${reduc_9_actuator_height/2}" radius="${wrist_diameter/2}" />
+				<cylinder length="${reduc_9_actuator_height/8}" radius="${wrist_diameter/4}" />
 			</geometry>
 			<origin rpy="0 0 0" xyz="0 0 0"/>
 		</collision>
 	</link>
-	<link name="end_effector">
-		<visual>
-			<geometry>
-				<cylinder length="${end_effector_height}" radius="${wrist_diameter/4}" />
-			</geometry>
-			<origin rpy="0 0 0" xyz="0 0 ${end_effector_height/2}"/>
-			<material name="thing"/>
-		</visual>
-		<collision>
-			<geometry>
-				<cylinder length="${reduc_9_actuator_height/2}" radius="${wrist_diameter/2}" />
+	<link name="right_differential">
+		<visual>
+			<geometry>
+				<cylinder length="${reduc_9_actuator_height/8}" radius="${wrist_diameter/4}" />
+			</geometry>
+			<origin rpy="0 0 0" xyz="0 0 0"/>
+			<material name="green"/>
+		</visual>
+		<collision>
+			<geometry>
+				<cylinder length="${reduc_9_actuator_height/8}" radius="${wrist_diameter/4}" />
 			</geometry>
 			<origin rpy="0 0 0" xyz="0 0 0"/>
@@ -200,11 +204,4 @@
 		<parent link="elbow_arm1"/>
 		<child link="elbow_arm2"/>
-	</joint>
-	<joint name="end_effector_join" type="fixed">
-		<origin xyz="${wrist_diameter/2} 0 0"
-				rpy="0 ${pi/2} 0"/>
-		<parent link="wrist"/>
-		<child link="end_effector"/>
-        <limit effort="30" velocity="1.0" lower="0" upper="${3.547/2.5 * pi}" />
 	</joint>
 	<!-- MOVING JOINTS -->
@@ -222,5 +219,5 @@
 		<parent link="waist"/>
 		<child link="shoulder"/>
-        <limit effort="30" velocity="1.0" lower="-${1.7}" upper="${2.42}" />
+        <limit effort="30" velocity="1.0" lower="-${2.57}" upper="${3.71}" />
 	</joint>
 	<joint name="elbow_joint" type="revolute">
@@ -232,11 +229,185 @@
         <limit effort="30" velocity="1.0" lower="0" upper="${2.28}" />
 	</joint>
-	<joint name="wrist_joint" type="revolute">
+	<joint name="left_differential_joint" type="revolute">
 		<origin xyz="${elbow_arm2_length} 0 -${arm_height/2}"
 				rpy="0 0 ${wrist_angle_offset}"/>
 		<axis rpy="0 0 0" xyz="0 0 1"/>
 		<parent link="elbow_arm2"/>
-		<child link="wrist"/>
-        <limit effort="30" velocity="1.0" lower="${-pi/2}" upper="${pi}" />
-	</joint>
+		<child link="left_differential"/>
+        <limit effort="30" velocity="1.0" lower="${-2*pi}" upper="${2*pi}"/>
+	</joint>
+	<joint name="right_differential_joint" type="revolute">
+		<origin xyz="${elbow_arm2_length} 0 ${arm_height/2}"
+				rpy="${pi} 0 ${wrist_angle_offset}"/>
+		<axis rpy="0 0 0" xyz="0 0 1"/>
+		<parent link="elbow_arm2"/>
+		<child link="right_differential"/>
+        <limit effort="30" velocity="1.0" lower="${-2*pi}" upper="${2*pi}"/>
+	</joint>
+	<!-- ROS2 CONTROL -->
+	<ros2_control name="pi3hat_hardware_interface" type="system">
+		<hardware>
+			<plugin>pi3hat_hardware_interface/Pi3HatHardwareInterface</plugin>
+				<param name="imu_mounting_deg.yaw">0</param>
+				<param name="imu_mounting_deg.pitch">0</param>
+				<param name="imu_mounting_deg.roll">0</param>
+				<param name="imu_sampling_rate">1000</param>
+				<param name="can_1_fdcan_frame">true</param>
+				<param name="can_1_automatic_retransmission">true</param>
+				<param name="can_1_bitrate_switch">true</param>
+				<param name="can_2_fdcan_frame">true</param>
+				<param name="can_2_automatic_retransmission">true</param>
+				<param name="can_2_bitrate_switch">true</param>
+				<param name="can_3_fdcan_frame">true</param>
+				<param name="can_3_automatic_retransmission">true</param>
+				<param name="can_3_bitrate_switch">true</param>
+				<param name="can_4_fdcan_frame">true</param>
+				<param name="can_4_automatic_retransmission">true</param>
+				<param name="can_4_bitrate_switch">true</param>
+				<param name="can_5_fdcan_frame">true</param>
+				<param name="can_5_automatic_retransmission">true</param>
+				<param name="can_5_bitrate_switch">true</param>
+		</hardware>
+		<joint name="waist_joint">
+			<param name="controller_type">moteus</param>
+			<param name="controller_can_bus">1</param>
+			<param name="controller_can_id">1</param>
+			<param name="motor_direction">1</param>
+			<param name="motor_position_offset">0.0</param>
+			<param name="motor_position_max">${pi *  waist_reduction_ratio}</param>
+			<param name="motor_position_min">${-pi * waist_reduction_ratio}</param>
+			<param name="motor_velocity_max">5.0</param>
+			<param name="motor_torque_max">1.0</param>
+			<command_interface name="position"/>
+			<command_interface name="velocity"/>
+			<command_interface name="effort"/>
+			<state_interface name = "position"/>
+			<state_interface name = "velocity"/>
+			<state_interface name = "effort"/>
+			<state_interface name = "temperature"/>
+		</joint>
+		<transmission name="waist_joint_transmission">
+            <plugin>transmission_interface/SimpleTransmission</plugin>
+            <actuator name="waist_actuator" role="actuator1"/>
+            <joint name="waist_joint" role="joint1">
+                <mechanical_reduction>${waist_reduction_ratio}</mechanical_reduction>
+                <offset>0</offset>
+            </joint>
+		</transmission>
+		<joint name="shoulder_joint">
+			<param name="controller_type">moteus</param>
+			<param name="controller_can_bus">2</param>
+			<param name="controller_can_id">2</param>
+			<param name="motor_direction">1</param>
+			<param name="motor_position_offset">0.0</param>
+			<param name="motor_position_max">${2.42 * shoulder_reduction_ratio}</param>
+			<param name="motor_position_min">${-1.7 * shoulder_reduction_ratio}</param>
+			<param name="motor_velocity_max">5.0</param>
+			<param name="motor_torque_max">1.0</param>
+			<command_interface name="position"/>
+			<command_interface name="velocity"/>
+			<command_interface name="effort"/>
+			<state_interface name = "position"/>
+			<state_interface name = "velocity"/>
+			<state_interface name = "effort"/>
+			<state_interface name = "temperature"/>
+		</joint>
+		<transmission name="shoulder_joint_transmission">
+            <plugin>transmission_interface/SimpleTransmission</plugin>
+            <actuator name="shoulder_actuator" role="actuator1"/>
+            <joint name="shoulder_joint" role="joint1">
+                <mechanical_reduction>${shoulder_reduction_ratio}</mechanical_reduction>
+                <offset>0</offset>
+            </joint>
+		</transmission>
+		<joint name="elbow_joint">
+			<param name="controller_type">moteus</param>
+			<param name="controller_can_bus">3</param>
+			<param name="controller_can_id">3</param>
+			<param name="motor_direction">1</param>
+			<param name="motor_position_offset">0.0</param>
+			<param name="motor_position_max">${2.28 * elbow_reduction_ratio}</param>
+			<param name="motor_position_min">${0.00 * elbow_reduction_ratio}</param>
+			<param name="motor_velocity_max">5.0</param>
+			<param name="motor_torque_max">1.0</param>
+			<command_interface name="position"/>
+			<command_interface name="velocity"/>
+			<command_interface name="effort"/>
+			<state_interface name = "position"/>
+			<state_interface name = "velocity"/>
+			<state_interface name = "effort"/>
+			<state_interface name = "temperature"/>
+		</joint>
+		<transmission name="elbow_joint_transmission">
+            <plugin>transmission_interface/SimpleTransmission</plugin>
+            <actuator name="elbow_actuator" role="actuator1"/>
+            <joint name="elbow_joint" role="joint1">
+                <mechanical_reduction>${elbow_reduction_ratio}</mechanical_reduction>
+                <offset>0</offset>
+            </joint>
+		</transmission>
+		<!-- WRIST TRANSMISSION WHICH IS DIFFERENTIAL -->
+		<joint name="left_differential_joint">
+			<param name="controller_type">moteus</param>
+			<param name="controller_can_bus">4</param>
+			<param name="controller_can_id">4</param>
+			<param name="motor_direction">1</param>
+			<param name="motor_position_offset">0.0</param>
+			<param name="motor_position_max">${2*pi * wrist_reduction_ratio}</param>
+			<param name="motor_position_min">${-2*pi * wrist_reduction_ratio}</param>
+			<param name="motor_velocity_max">10.0</param>
+			<param name="motor_torque_max">5.0</param>
+			<command_interface name="position"/>
+			<command_interface name="velocity"/>
+			<command_interface name="effort"/>
+			<state_interface name="position"/>
+			<state_interface name="velocity"/>
+			<state_interface name="effort"/>
+			<state_interface name="temperature"/>
+		</joint>
+		<joint name="right_differential_joint">
+			<param name="controller_type">moteus</param>
+			<param name="controller_can_bus">5</param>
+			<param name="controller_can_id">5</param>
+			<param name="motor_direction">-1</param>
+			<param name="motor_position_offset">0.0</param>
+			<param name="motor_position_max">${2*pi * wrist_reduction_ratio}</param>
+			<param name="motor_position_min">${-2*pi * wrist_reduction_ratio}</param>
+			<param name="motor_velocity_max">10.0</param>
+			<param name="motor_torque_max">5.0</param>
+			<command_interface name="position"/>
+			<command_interface name="velocity"/>
+			<command_interface name="effort"/>
+			<state_interface name="position"/>
+			<state_interface name="velocity"/>
+			<state_interface name="effort"/>
+			<state_interface name="temperature"/>
+		</joint>
+		<!-- Differential Transmission -->
+		<transmission name="differential_drive_transmission">
+			<plugin>transmission_interface/DifferentialTransmission</plugin>
+			<actuator name="left_differential_actuator" role="actuator1"/>
+			<actuator name="right_differential_actuator" role="actuator2"/>
+			<joint name="left_differential_joint" role="joint1">
+				<mechanical_reduction>${wrist_reduction_ratio}</mechanical_reduction>
+				<offset>0.0</offset>
+			</joint>
+			<joint name="right_differential_joint" role="joint2">
+				<mechanical_reduction>${wrist_reduction_ratio}</mechanical_reduction>
+				<offset>0.0</offset>
+			</joint>
+		</transmission>
+		<sensor name="imu_sensor">
+			<state_interface name = "orientation.x"/>
+			<state_interface name = "orientation.y"/>
+			<state_interface name = "orientation.z"/>
+			<state_interface name = "orientation.w"/>
+			<state_interface name = "angular_velocity.x"/>
+			<state_interface name = "angular_velocity.y"/>
+			<state_interface name = "angular_velocity.z"/>
+			<state_interface name = "linear_acceleration.x"/>
+			<state_interface name = "linear_acceleration.y"/>
+			<state_interface name = "linear_acceleration.z"/>
+		</sensor>
+	</ros2_control>
 </robot>

Commit message: Properly modeled wrist differential(hopefully) in rviz + real

File: test/urdf/myrobot.urdf.xacro (robot description, xacro)
@@ -20,5 +20,5 @@
 	<xacro:property name="wrist_angle_offset" value="${-pi/4 - elbow_arm1_angle_offset}"/>
 	<xacro:property name="wrist_diameter" value="${0.04 * multiplier}"/>
-	<xacro:property name="end_effector_height" value="${0.04 * multiplier}"/>
+	<xacro:property name="end_effector_rod_len" value="${0.05 * multiplier}"/>
 	<material name="black">
 		<color rgba="0 0 0 1"/>
@@ -153,14 +153,14 @@
 		<visual>
 			<geometry>
+				<cylinder length="${end_effector_rod_len}" radius="${wrist_diameter/8}" />
+			</geometry>
+			<origin rpy="0 0 0" xyz="0 0 ${end_effector_rod_len/2}"/>
+			<material name="green"/>
+		</visual>
+		<collision>
+			<geometry>
 				<cylinder length="${reduc_9_actuator_height/8}" radius="${wrist_diameter/4}" />
 			</geometry>
 			<origin rpy="0 0 0" xyz="0 0 0"/>
-			<material name="green"/>
-		</visual>
-		<collision>
-			<geometry>
-				<cylinder length="${reduc_9_actuator_height/8}" radius="${wrist_diameter/4}" />
-			</geometry>
-			<origin rpy="0 0 0" xyz="0 0 0"/>
 		</collision>
 	</link>
@@ -168,5 +168,5 @@
 		<visual>
 			<geometry>
-				<cylinder length="${reduc_9_actuator_height/8}" radius="${wrist_diameter/4}" />
+				<cylinder length="${reduc_9_actuator_height/2}" radius="${wrist_diameter/4}" />
 			</geometry>
 			<origin rpy="0 0 0" xyz="0 0 0"/>
@@ -229,18 +229,20 @@
         <limit effort="30" velocity="1.0" lower="0" upper="${2.28}" />
 	</joint>
-	<joint name="left_differential_joint" type="revolute">
-		<origin xyz="${elbow_arm2_length} 0 -${arm_height/2}"
-				rpy="0 0 ${wrist_angle_offset}"/>
-		<axis rpy="0 0 0" xyz="0 0 1"/>
-		<parent link="elbow_arm2"/>
-		<child link="left_differential"/>
-        <limit effort="30" velocity="1.0" lower="${-2*pi}" upper="${2*pi}"/>
-	</joint>
+	<!-- Technically the PITCH of wrist -->
 	<joint name="right_differential_joint" type="revolute">
-		<origin xyz="${elbow_arm2_length} 0 ${arm_height/2}"
-				rpy="${pi} 0 ${wrist_angle_offset}"/>
-		<axis rpy="0 0 0" xyz="0 0 1"/>
+		<origin xyz="${elbow_arm2_length} 0 0"
+				rpy="${-pi} 0 ${wrist_angle_offset}"/>
+		<axis rpy="0 0 0" xyz="0 0 -1"/>
 		<parent link="elbow_arm2"/>
 		<child link="right_differential"/>
+        <limit effort="30" velocity="1.0" lower="${-2*pi}" upper="${2*pi}"/>
+	</joint>
+	<!-- Technically the ROLL of wrist -->
+	<joint name="left_differential_joint" type="revolute">
+		<origin xyz="0 0 0"
+				rpy="${pi/2} 0 0"/>
+		<axis rpy="0 0 0" xyz="0 0 1"/>
+		<parent link="right_differential"/>
+		<child link="left_differential"/>
         <limit effort="30" velocity="1.0" lower="${-2*pi}" upper="${2*pi}"/>
 	</joint>
@@ -390,9 +392,9 @@
 			<actuator name="right_differential_actuator" role="actuator2"/>
 			<joint name="left_differential_joint" role="joint1">
-				<mechanical_reduction>${wrist_reduction_ratio}</mechanical_reduction>
+				<mechanical_reduction>${wrist_reduction_ratio / 2}</mechanical_reduction>
 				<offset>0.0</offset>
 			</joint>
 			<joint name="right_differential_joint" role="joint2">
-				<mechanical_reduction>${wrist_reduction_ratio}</mechanical_reduction>
+				<mechanical_reduction>${wrist_reduction_ratio / 2}</mechanical_reduction>
 				<offset>0.0</offset>
 			</joint>

Commit message: Proper FK and actual more-accurate modeling for myrobot urdf

File: test/urdf/myrobot.urdf.xacro (robot description, xacro)
@@ -42,5 +42,5 @@
 		<color rgba="0.2 0.7 0.4 1"/>
 	</material>
-	<link name="world" />
+	<link name="base_link" />
 	<!-- LINKS -->
 	<link name="waist">
@@ -180,4 +180,5 @@
 		</collision>
 	</link>
+	<link name="end_effector" />
 	<!-- MODELING JOINTS -->
 	<joint name="waist_arm_join" type="fixed">
@@ -205,9 +206,15 @@
 		<child link="elbow_arm2"/>
 	</joint>
+	<joint name="end_effector_join" type="fixed">
+		<origin xyz="0 0 ${end_effector_rod_len}"
+				rpy="0 0 0"/>
+		<parent link="left_differential"/>
+		<child link="end_effector"/>
+	</joint>
 	<!-- MOVING JOINTS -->
 	<joint name="waist_joint" type="revolute">
 		<origin xyz="0 0 ${reduc_9_actuator_height}"/>
 		<axis rpy="0 0 0" xyz="0 0 1"/>
-		<parent link="world"/>
+		<parent link="base_link"/>
 		<child link="waist"/>
         <limit effort="30" velocity="1.0" lower="-${pi}" upper="${pi}" />
@@ -231,5 +238,5 @@
 	<!-- Technically the PITCH of wrist -->
 	<joint name="right_differential_joint" type="revolute">
-		<origin xyz="${elbow_arm2_length} 0 0"
+		<origin xyz="${elbow_arm2_length} 0 -${elbow_arm_width/2}"
 				rpy="${-pi} 0 ${wrist_angle_offset}"/>
 		<axis rpy="0 0 0" xyz="0 0 -1"/>

Commit message: Fixing order of control for differential wrist and some new scripts for zeroing

File: test/urdf/myrobot.urdf.xacro (robot description, xacro)
@@ -238,5 +238,5 @@
 	<!-- Technically the PITCH of wrist -->
 	<joint name="right_differential_joint" type="revolute">
-		<origin xyz="${elbow_arm2_length} 0 -${elbow_arm_width/2}"
+		<origin xyz="${elbow_arm2_length} 0 -${reduc_9_actuator_height/4}"
 				rpy="${-pi} 0 ${wrist_angle_offset}"/>
 		<axis rpy="0 0 0" xyz="0 0 -1"/>

Commit message: Actual proper modeling of bot + proper 0

File: test/urdf/myrobot.urdf.xacro (robot description, xacro)
@@ -5,20 +5,22 @@
 	<xacro:property name="reduc_9_actuator_height" value="${0.058 * multiplier}"/>
 	<xacro:property name="waist_reduction_ratio" value="9"/>
+	<xacro:property name="waist_height" value="${0.085 * multiplier}"/>
 	<xacro:property name="waist_arm_height" value="${0.01 * multiplier}"/>
 	<xacro:property name="shoulder_reduction_ratio" value="9"/>
-	<xacro:property name="shoulder_arm_angle_offset" value="${-0.5*pi - 0.52/4.5*pi}"/>
+	<xacro:property name="shoulder_arm_angle_offset" value="${-0.5*pi+0.8/4.5*pi}"/>
 	<xacro:property name="shoulder_arm_length" value="${0.1385 * multiplier}"/>
 	<xacro:property name="shoulder_arm_width" value="${0.047 * multiplier}"/>
 	<xacro:property name="arm_height" value="${0.03 * multiplier}"/>
 	<xacro:property name="elbow_reduction_ratio" value="5"/>
-	<xacro:property name="elbow_arm1_angle_offset" value="${-pi/6 + 0.15/2.5*pi}"/>
+	<xacro:property name="elbow_arm1_angle_offset" value="${0}"/>
 	<xacro:property name="elbow_arm2_angle_offset" value="-${pi/4}"/>
 	<xacro:property name="elbow_arm1_length" value="${0.065 * multiplier}"/>
 	<xacro:property name="elbow_arm2_length" value="${0.110 * multiplier}"/>
 	<xacro:property name="elbow_arm_width" value="${0.020 * multiplier}"/>
+	<xacro:property name="right_differential_diameter" value="${0.045 * multiplier}"/>
 	<xacro:property name="wrist_reduction_ratio" value="6"/>
-	<xacro:property name="wrist_angle_offset" value="${-pi/4 - elbow_arm1_angle_offset}"/>
+	<xacro:property name="wrist_angle_offset" value="${-pi/2-0.20}"/>
 	<xacro:property name="wrist_diameter" value="${0.04 * multiplier}"/>
-	<xacro:property name="end_effector_rod_len" value="${0.05 * multiplier}"/>
+	<xacro:property name="end_effector_rod_len" value="${0.100 * multiplier}"/>
 	<material name="black">
 		<color rgba="0 0 0 1"/>
@@ -47,29 +49,14 @@
 		<visual>
 			<geometry>
-				<cylinder length="${reduc_9_actuator_height}" radius="${reduc_9_actuator_diameter/2}" />
-			</geometry>
-			<origin rpy="0 0 0" xyz="0 0 -${reduc_9_actuator_height/2}"/>
+				<cylinder length="${waist_height}" radius="${reduc_9_actuator_diameter/2}" />
+			</geometry>
+			<origin rpy="0 0 0" xyz="0 0 -${waist_height/2}"/>
 			<material name="orange"/>
 		</visual>
 		<collision>
 			<geometry>
-				<cylinder length="${reduc_9_actuator_height}" radius="${reduc_9_actuator_diameter/2}" />
-			</geometry>
-			<origin rpy="0 0 0" xyz="0 0 -${reduc_9_actuator_height/2}"/>
-		</collision>
-	</link>
-	<link name="waist_arm">
-		<visual>
-			<geometry>
-				<cylinder radius="${reduc_9_actuator_diameter/2}" length="${waist_arm_height}"/>
-			</geometry>
-			<origin rpy="0 0 0" xyz="0 0 ${waist_arm_height/2}"/>
-			<material name="black"/>
-		</visual>
-		<collision>
-			<geometry>
-				<box size="${reduc_9_actuator_diameter} ${reduc_9_actuator_diameter} ${waist_arm_height}" />
-			</geometry>
-			<origin rpy="0 0 0" xyz="0 0 ${waist_arm_height/2}"/>
+				<cylinder length="${waist_height}" radius="${reduc_9_actuator_diameter/2}" />
+			</geometry>
+			<origin rpy="0 0 0" xyz="0 0 -${waist_height/2}"/>
 		</collision>
 	</link>
@@ -168,5 +155,5 @@
 		<visual>
 			<geometry>
-				<cylinder length="${reduc_9_actuator_height/2}" radius="${wrist_diameter/4}" />
+				<cylinder length="${reduc_9_actuator_height/2}" radius="${right_differential_diameter/2}" />
 			</geometry>
 			<origin rpy="0 0 0" xyz="0 0 0"/>
@@ -182,10 +169,4 @@
 	<link name="end_effector" />
 	<!-- MODELING JOINTS -->
-	<joint name="waist_arm_join" type="fixed">
-		<origin xyz="0 0 0"
-				rpy="0 0 0"/>
-		<parent link="waist"/>
-		<child link="waist_arm"/>
-	</joint>
 	<joint name="shoulder_arm_join" type="fixed">
 		<origin xyz="0 0 0"
@@ -196,5 +177,5 @@
 	<joint name="elbow_arm_join" type="fixed">
 		<origin xyz="0 0 ${arm_height/2}"
-				rpy="0 0 ${elbow_arm1_angle_offset}"/>
+				rpy="0 0 ${-1.27/2.5*pi}"/>
 		<parent link="elbow"/>
 		<child link="elbow_arm1"/>
@@ -214,5 +195,5 @@
 	<!-- MOVING JOINTS -->
 	<joint name="waist_joint" type="revolute">
-		<origin xyz="0 0 ${reduc_9_actuator_height}"/>
+		<origin xyz="0 0 ${waist_height}"/>
 		<axis rpy="0 0 0" xyz="0 0 1"/>
 		<parent link="base_link"/>
@@ -221,5 +202,5 @@
 	</joint>
 	<joint name="shoulder_joint" type="revolute">
-		<origin xyz="0 0 ${waist_arm_height + reduc_9_actuator_diameter/2}"
+		<origin xyz="0 0 ${reduc_9_actuator_diameter/2}"
 				rpy="-${pi/2} 0 0"/>
 		<axis rpy="0 0 0" xyz="0 0 1"/>
@@ -230,5 +211,5 @@
 	<joint name="elbow_joint" type="revolute">
 		<origin xyz="${cos(shoulder_arm_angle_offset) * shoulder_arm_length} ${sin(shoulder_arm_angle_offset) * shoulder_arm_length} 0"
-				rpy="${pi} 0 0"/>
+				rpy="${pi} 0 ${shoulder_arm_angle_offset}"/>
 		<axis rpy="0 0 0" xyz="0 0 1"/>
 		<parent link="shoulder"/>
